File: PlaybackSection/PlaybackSection.kicad_pcb (KiCad board)
At the start: 2 copper layers, 162.7 x 250.1 mm, 22 parts, among them SW1 RotaryEncoder, SW2 RotaryEncoder, SW3 RotaryEncoder, SW4 RotaryEncoder, SW5 RotaryEncoder, SW6 RotaryEncoder, SW7 RotaryEncoder, SW8 RotaryEncoder, U1 TLC5947DAP, U2 MCP23017x-x-SS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

Commit message: continued wiring for tlc5947 and mcp23017
Parts:
- removed the REF** at (206.0, 53.3)
- moved U2 133.2 mm to (147.1, 86.6)
- moved D5 5.96 mm to (159.3, 99.6)
- moved U3 3.59 mm to (35.8, 25.1)
Connections:
- A1 pad 13: Net-(A1-GND-Pad13) -> GND
- A1 pad 18: Net-(A1-GND-Pad13) -> GND
- A1 pad 21: unconnected-(A1-GPIO16-Pad21) -> Net-(A1-GPIO16)
- A1 pad 22: unconnected-(A1-GPIO17-Pad22) -> Net-(A1-GPIO17)
- A1 pad 23: Net-(A1-GND-Pad13) -> GND
- A1 pad 24: unconnected-(A1-GPIO18-Pad24) -> Net-(A1-GPIO18)
- A1 pad 25: unconnected-(A1-GPIO19-Pad25) -> Net-(A1-GPIO19)
- A1 pad 28: Net-(A1-GND-Pad13) -> GND
- A1 pad 3: Net-(A1-GND-Pad13) -> GND
- A1 pad 33: unconnected-(A1-AGND-Pad33) -> GND
- A1 pad 36: unconnected-(A1-3V3-Pad36) -> +3V3
- A1 pad 38: Net-(A1-GND-Pad13) -> GND
- A1 pad 8: Net-(A1-GND-Pad13) -> GND
- SW1 pad A: unconnected-(SW1-PadA) -> Net-(U2-GPB0)
- SW1 pad B: unconnected-(SW1-PadB) -> Net-(U2-GPB1)
- SW1 pad C: unconnected-(SW1-PadC) -> GND
- SW2 pad A: unconnected-(SW2-PadA) -> Net-(U2-GPB2)
- SW2 pad B: unconnected-(SW2-PadB) -> Net-(U2-GPB3)
- SW2 pad C: unconnected-(SW2-PadC) -> GND
- SW3 pad A: unconnected-(SW3-PadA) -> Net-(U2-GPB4)
- SW3 pad B: unconnected-(SW3-PadB) -> Net-(U2-GPB5)
- SW3 pad C: unconnected-(SW3-PadC) -> GND
- SW4 pad A: unconnected-(SW4-PadA) -> Net-(U2-GPB6)
- SW4 pad B: unconnected-(SW4-PadB) -> Net-(U2-GPB7)
- SW4 pad C: unconnected-(SW4-PadC) -> GND
- SW5 pad A: unconnected-(SW5-PadA) -> Net-(U2-GPA7)
- SW5 pad B: unconnected-(SW5-PadB) -> Net-(U2-GPA6)
- SW5 pad C: unconnected-(SW5-PadC) -> GND
- SW6 pad A: unconnected-(SW6-PadA) -> Net-(U2-GPA5)
- SW6 pad B: unconnected-(SW6-PadB) -> Net-(U2-GPA4)
- SW6 pad C: unconnected-(SW6-PadC) -> GND
- SW7 pad A: unconnected-(SW7-PadA) -> Net-(U2-GPA3)
- SW7 pad B: unconnected-(SW7-PadB) -> Net-(U2-GPA2)
- SW7 pad C: unconnected-(SW7-PadC) -> GND
- SW8 pad A: unconnected-(SW8-PadA) -> Net-(U2-GPA1)
- SW8 pad B: unconnected-(SW8-PadB) -> Net-(U2-GPA0)
- SW8 pad C: unconnected-(SW8-PadC) -> GND
- U1 pad 1: unconnected-(U1-GND-Pad1) -> GND
- U1 pad 2: unconnected-(U1-BLANK-Pad2) -> Net-(A1-GPIO16)
- U1 pad 3: unconnected-(U1-SCLK-Pad3) -> Net-(A1-GPIO18)
- U1 pad 30: unconnected-(U1-XLAT-Pad30) -> Net-(A1-GPIO17)
- U1 pad 31: unconnected-(U1-IREF-Pad31) -> Net-(U1-IREF)
- U1 pad 32: unconnected-(U1-VCC-Pad32) -> +3V3
- U1 pad 33: unconnected-(U1-PowerPAD-Pad33) -> GND
- U1 pad 4: unconnected-(U1-SIN-Pad4) -> Net-(A1-GPIO19)
- U2 pad 1: unconnected-(U2-GPB0-Pad1) -> Net-(U2-GPB0)
- U2 pad 10: unconnected-(U2-V_{SS}-Pad10) -> GND
- U2 pad 15: unconnected-(U2-A0-Pad15) -> GND
- U2 pad 16: unconnected-(U2-A1-Pad16) -> GND
- U2 pad 17: unconnected-(U2-A2-Pad17) -> GND
- U2 pad 2: unconnected-(U2-GPB1-Pad2) -> Net-(U2-GPB1)
- U2 pad 21: unconnected-(U2-GPA0-Pad21) -> Net-(U2-GPA0)
- U2 pad 22: unconnected-(U2-GPA1-Pad22) -> Net-(U2-GPA1)
- U2 pad 23: unconnected-(U2-GPA2-Pad23) -> Net-(U2-GPA2)
- U2 pad 24: unconnected-(U2-GPA3-Pad24) -> Net-(U2-GPA3)
- U2 pad 25: unconnected-(U2-GPA4-Pad25) -> Net-(U2-GPA4)
- U2 pad 26: unconnected-(U2-GPA5-Pad26) -> Net-(U2-GPA5)
- U2 pad 27: unconnected-(U2-GPA6-Pad27) -> Net-(U2-GPA6)
- U2 pad 28: unconnected-(U2-GPA7-Pad28) -> Net-(U2-GPA7)
- U2 pad 3: unconnected-(U2-GPB2-Pad3) -> Net-(U2-GPB2)
- U2 pad 4: unconnected-(U2-GPB3-Pad4) -> Net-(U2-GPB3)
- U2 pad 5: unconnected-(U2-GPB4-Pad5) -> Net-(U2-GPB4)
- U2 pad 6: unconnected-(U2-GPB5-Pad6) -> Net-(U2-GPB5)
- U2 pad 7: unconnected-(U2-GPB6-Pad7) -> Net-(U2-GPB6)
- U2 pad 8: unconnected-(U2-GPB7-Pad8) -> Net-(U2-GPB7)
- U2 pad 9: unconnected-(U2-V_{DD}-Pad9) -> +3V3
- U3 pad 9: unconnected-(U3-V_{DD}-Pad9) -> +3V3
