File: PlaybackSection/PlaybackSection.kicad_sch (KiCad schematic)
At the start: 19 parts, among them SW1 RotaryEncoder, SW2 RotaryEncoder, SW3 RotaryEncoder, SW4 RotaryEncoder, SW5 RotaryEncoder, SW6 RotaryEncoder, SW7 RotaryEncoder, SW8 RotaryEncoder, U1 TLC5947DAP, U2 MCP23017x-x-SS, U3 MCP23017x-x-SS, U4 MCP23017x-x-SS, U5 TB6612FNG

Commit message: continued wiring for tlc5947 and mcp23017
Parts:
- added R1: R, symbol Device:R
Connections:
- net GND: now also A1.13 (GND), A1.18 (GND), A1.23 (GND), A1.28 (GND), A1.3 (GND), A1.33 (AGND), A1.38 (GND), A1.8 (GND), SW1.C, SW2.C, SW3.C, SW4.C, SW5.C, SW6.C, SW7.C, SW8.C, U1.1 (GND), U1.33 (PowerPAD), U2.10 (V_{SS}), U2.15 (A0), U2.16 (A1), U2.17 (A2), R1.2
- net at SW5.A: now also U2.28 (GPA7)
- net at SW5.B: now also U2.27 (GPA6)
- net at SW6.A: now also U2.26 (GPA5)
- net at SW6.B: now also U2.25 (GPA4)
- net at SW4.A: now also U2.7 (GPB6)
- net at SW4.B: now also U2.8 (GPB7)
- net at SW1.A: now also U2.1 (GPB0)
- net at SW1.B: now also U2.2 (GPB1)
- net +3V3: now reaches U3.9 (V_{DD})
- net +3V3: now also A1.36 (3V3), U1.32 (VCC), U2.9 (V_{DD})
- net at SW7.A: now also U2.24 (GPA3)
- net at SW7.B: now also U2.23 (GPA2)
- net at U1.2 (BLANK): now also A1.21 (GPIO16)
- net at U1.3 (SCLK): now also A1.24 (GPIO18)
- net at U1.30 (XLAT): now also A1.22 (GPIO17)
- net at U1.31 (IREF): now also R1.1
- net at U1.4 (SIN): now also A1.25 (GPIO19)
- net at SW3.A: now also U2.5 (GPB4)
- net at SW3.B: now also U2.6 (GPB5)
- net at SW2.A: now also U2.3 (GPB2)
- net at SW2.B: now also U2.4 (GPB3)
- net at SW8.A: now also U2.22 (GPA1)
- net at SW8.B: now also U2.21 (GPA0)
- no-connect marks 1 -> 2
Other:
- moved on the sheet: A1, D1, D2, D3, D4, D5, SW1, SW2, SW3, SW4, SW5, SW6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
